File: XuLabPlatform.kicad_pcb (KiCad board)
At the start: 4 copper layers, 115 x 123 mm, 75 parts, among them J1 SWD Connector, J10 Servo7, J11 Servo8, J12 Thruster SGN, J13 USB_B_Micro, J14 CAN, J15 I2C, J16 UART, J2 Conn_01x04, J3 1986660-2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

Commit message: Change pressure connector from JST-GH-BM04B to JST-GH-SM04B
Parts:
- J10: value Servo7 -> Servo
- J11: value Servo8 -> Servo
- J12: value Thruster SGN -> Thruster
- J2: footprint Connector_JST:JST_GH_BM04B-GHS-TBT_1x04-1MP_P1.25mm_Vertical -> Connector_JST:JST_GH_SM04B-GHS-TB_1x04-1MP_P1.25mm_Horizontal
- J4: value Servo1 -> Servo
- J5: value Servo2 -> Servo
- J6: value Servo3 -> Servo
- J7: value Servo4 -> Servo
- J8: value Servo5 -> Servo
- J9: value Servo6 -> Servo
- moved C17 0.25 mm to (105.5, 44.8), turned to 180 degrees
- turned J2 to 180 degrees
Routing:
- net GND: track 129.1 -> 127.6 mm
- net +3.3V: track 58.2 -> 57.0 mm
- net /I2C1_SDA: track 81.7 -> 82.6 mm
- net /I2C1_SCL: track 82.8 -> 82.0 mm, vias 0 -> 2
