File: Project/Controller/Microcontroller.kicad_sch (KiCad schematic)
At the start: 38 parts, among them J2 SWD, J3 USB_C_Receptacle_USB2.0_16P, SW1 SW_SPDT, SW2 SW_SPDT, SW3 SW_Push, U4 STM32F446RCTx, U5 24AA64-OT, U6 USBLC6-2SC6, Y1 8MHz

Commit message: Re-annotate symbols
Parts:
- renumbered C31 to C18, C18 to C19, C19 to C20, R17 to R10, R12 to R11, R13 to R12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
