File: Project/Controller/Power.kicad_sch (KiCad schematic)
At the start: 15 parts, among them J1 Power, U1 LM66100DCK, U2 MIC5219-3.3YM5, U3 LM66100DCK

Commit message: Change power connector to JST GH
Parts:
- J1: footprint Connector_JST:JST_XH_S2B-XH-A_1x02_P2.50mm_Horizontal -> Connector_JST:JST_GH_SM02B-GHS-TB_1x02-1MP_P1.25mm_Horizontal; Listing https://www.digikey.com/en/products/detail/jst-sales-america-inc/S2B-XH-A/1651055 -> https://www.digikey.com/en/products/detail/jst-sales-america-inc/SM02B-GHS-TB/807786
Changed lines of the file:
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@@
 			)
 		)
-		(property "Footprint" "Connector_JST:JST_XH_S2B-XH-A_1x02_P2.50mm_Horizontal"
+		(property "Footprint" "Connector_JST:JST_GH_SM02B-GHS-TB_1x02-1MP_P1.25mm_Horizontal"
 			(at 58.42 50.8 0)
 			(effects
@@
 			)
 		)
-		(property "Datasheet" "https://www.jst-mfg.com/product/pdf/eng/eXH.pdf"
+		(property "Datasheet" "https://www.jst.com/wp-content/uploads/2025/06/eGH.pdf"
 			(at 58.42 50.8 0)
 			(effects
@@
 			)
 		)
-		(property "Listing" "https://www.digikey.com/en/products/detail/jst-sales-america-inc/S2B-XH-A/1651055"
+		(property "Listing" "https://www.digikey.com/en/products/detail/jst-sales-america-inc/SM02B-GHS-TB/807786"
 			(at 58.42 50.8 0)
 			(effects

Commit message: Add power test points
Parts:
- added TP1: Power, TestPoint:TestPoint_2Pads_Pitch2.54mm_Drill0.8mm, symbol Connector:TestPoint_2Pole
Connections:
- net +3.3V: now also TP1.1
- net GND: now also TP1.2
Changed lines of the file:
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@@
+	(wire
+		(pts
+			(xy 88.9 114.3) (xy 88.9 115.57)
+		)
+		(stroke
+			(width 0)
+			(type default)
+		)
+	)
 	(wire
 		(pts
@@
 		(pts
 			(xy 95.25 66.04) (xy 101.6 66.04)
+		)
+		(stroke
+			(width 0)
+			(type default)
+		)
+	)
+	(wire
+		(pts
+			(xy 88.9 125.73) (xy 88.9 127)
 		)
 		(stroke
@@
 	)
 	(symbol
+		(lib_id "power:GND")
+		(at 88.9 127 0)
+		(unit 1)
+		(exclude_from_sim no)
+		(in_bom yes)
+		(on_board yes)
+		(dnp no)
+		(fields_autoplaced yes)
+		(property "Reference" "#PWR091"
+			(at 88.9 133.35 0)
+			(effects
+				(font
+					(size 1.27 1.27)
+				)
+				(hide yes)
+			)
+		)
+		(property "Value" "GND"
+			(at 91.44 128.2699 0)
+			(effects
+				(font
+					(size 1.27 1.27)
+				)
+				(justify left)
+			)
+		)
+		(property "Footprint" ""
+			(at 88.9 127 0)
+			(effects
+				(font
+					(size 1.27 1.27)
+				)
+				(hide yes)
+			)
+		)
+		(property "Datasheet" ""
+			(at 88.9 127 0)
+			(effects
+				(font
+					(size 1.27 1.27)
+				)
+				(hide yes)
+			)
+		)
+		(property "Description" "Power symbol creates a global label with name \"GND\" , ground"
+			(at 88.9 127 0)
+			(effects
+				(font
+					(size 1.27 1.27)
+				)
+				(hide yes)
+			)
+		)
+		(pin "1"
+		)
+		(instances
+			(project "XuLabController"
+				(path "/71bb14ae-b730-4d22-a41d-cf68989dae2d/abfe70fc-8fea-4ce2-8a39-f4567326826d"
+					(reference "#PWR091")
+					(unit 1)
+				)
+			)
+		)
+	)
+	(symbol
 		(lib_id "power:+3.3V")
 		(at 215.9 60.96 0)
@@
 				(path "/71bb14ae-b730-4d22-a41d-cf68989dae2d/abfe70fc-8fea-4ce2-8a39-f4567326826d"
 					(reference "R2")
+					(unit 1)
+				)
+			)
+		)
+	)
+	(symbol
+		(lib_id "Connector:TestPoint_2Pole")
+		(at 88.9 120.65 270)
+		(unit 1)
+		(exclude_from_sim no)
+		(in_bom no)
+		(on_board yes)
+		(dnp no)
+		(fields_autoplaced yes)
+		(property "Reference" "TP1"
+			(at 91.44 119.3799 90)
+			(effects
+				(font
+					(size 1.27 1.27)
+				)
+				(justify left)
+			)
+		)
+		(property "Value" "Power"
+			(at 91.44 121.9199 90)
+			(effects
+				(font
+					(size 1.27 1.27)
+				)
+				(justify left)
+			)
+		)
+		(property "Footprint" "TestPoint:TestPoint_2Pads_Pitch2.54mm_Drill0.8mm"
+			(at 88.9 120.65 0)
+			(effects
+				(font
+					(size 1.27 1.27)
+				)
+				(hide yes)
+			)
+		)
+		(property "Datasheet" "None"
+			(at 88.9 120.65 0)
+			(effects
+				(font
+					(size 1.27 1.27)
+				)
+				(hide yes)
+			)
+		)
+		(property "Description" "2-polar test point"
+			(at 88.9 120.65 0)
+			(effects
+				(font
+					(size 1.27 1.27)
+				)
+				(hide yes)
+			)
+		)
+		(property "Listing" "None"
+			(at 88.9 120.65 0)
+			(effects
+				(font
+					(size 1.27 1.27)
+				)
+				(hide yes)
+			)
+		)
+		(property "Interchangeable" "N/A"
+			(at 88.9 120.65 0)
+			(effects
+				(font
+					(size 1.27 1.27)
+				)
+				(hide yes)
+			)
+		)
+		(pin "1"
+		)
+		(pin "2"
+		)
+		(instances
+			(project ""
+				(path "/71bb14ae-b730-4d22-a41d-cf68989dae2d/abfe70fc-8fea-4ce2-8a39-f4567326826d"
+					(reference "TP1")
 					(unit 1)
 				)
@@
 					(unit 1)
 				)
+			)
+		)
+	)
+	(symbol
+		(lib_id "power:+3.3V")
+		(at 88.9 114.3 0)
+		(unit 1)
+		(exclude_from_sim no)
+		(in_bom yes)
+		(on_board yes)
+		(dnp no)
+		(fields_autoplaced yes)
+		(property "Reference" "#PWR090"
+			(at 88.9 118.11 0)
+			(effects
+				(font
+					(size 1.27 1.27)
+				)
+				(hide yes)
+			)
+		)
+		(property "Value" "+3.3V"
+			(at 91.44 113.0299 0)
+			(effects
+				(font
+					(size 1.27 1.27)
+				)
+				(justify left)
+			)
+		)
+		(property "Footprint" ""
+			(at 88.9 114.3 0)
+			(effects
+				(font
+					(size 1.27 1.27)
+				)
+				(hide yes)
+			)
+		)
+		(property "Datasheet" ""
+			(at 88.9 114.3 0)
+			(effects
+				(font
+					(size 1.27 1.27)
+				)
+				(hide yes)
+			)
+		)
+		(property "Description" "Power symbol creates a global label with name \"+3.3V\""
+			(at 88.9 114.3 0)
+			(effects
+				(font
+					(size 1.27 1.27)
+				)
+				(hide yes)
+			)
+		)
+		(pin "1"
+		)
+		(instances
+			(project "XuLabController"
+				(path "/71bb14ae-b730-4d22-a41d-cf68989dae2d/abfe70fc-8fea-4ce2-8a39-f4567326826d"
+					(reference "#PWR090")
+					(unit 1)
+				)

Commit message: Add two more LEDs and increase LED series resistance
Parts:
- D2: value LED -> Red; Listing https://www.digikey.com/en/products/detail/liteon/LTST-C190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 -> https://www.digikey.com/en/products/detail/w%C3%BCrth-elekt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
- R3: value 75 -> 330; Listing https://www.digikey.com/en/products/detail/yageo/RC0402JR-0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 -> https://www.digikey.com/en/products/detail/yageo/RC0402FR-0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
Changed lines of the file:
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@@
 	(title_block
 		(title "Power")
-		(date "2026-02-05")
+		(date "2026-02-09")
 		(rev "B")
 		(company "CU Boulder Senior Design Team 29 - Xu Lab")
@@
 			)
 		)
-		(property "Value" "LED"
+		(property "Value" "Red"
 			(at 67.31 122.2374 90)
 			(effects
@@
 			)
 		)
-		(property "Datasheet" "https://optoelectronics.liteon.com/upload/download/DS-22-99-0151/LTST-C190KRKT.pdf"
+		(property "Datasheet" "https://www.we-online.com/components/products/datasheet/150060RS75000.pdf"
 			(at 63.5 119.38 0)
 			(effects
@@
 			)
 		)
-		(property "Listing" "https://www.digikey.com/en/products/detail/liteon/LTST-C190KRKT/386817"
+		(property "Listing" "https://www.digikey.com/en/products/detail/w%C3%BCrth-elektronik/150060RS75000/4489901"
 			(at 63.5 119.38 90)
 			(effects
@@
 			)
 		)
-		(property "Value" "75"
+		(property "Value" "330"
 			(at 66.04 129.5399 0)
 			(effects
@@
 			)
 		)
-		(property "Datasheet" "https://www.yageogroup.com/content/datasheet/asset/file/PYU-RC_GROUP_51_ROHS_L"
+		(property "Datasheet" "https://yageogroup.com/content/datasheet/asset/file/PYU-RC_GROUP_51_ROHS_L"
 			(at 63.5 128.27 0)
 			(effects
@@
 			)
 		)
-		(property "Listing" "https://www.digikey.com/en/products/detail/yageo/RC0402JR-0775RL/726505"
+		(property "Listing" "https://www.digikey.com/en/products/detail/yageo/RC0402FR-07330RL/726594"
 			(at 63.5 128.27 0)
 			(effects

Commit message: Change 0402 footprints to 0603
Parts:
- R3: footprint Resistor_SMD:R_0402_1005Metric -> Resistor_SMD:R_0603_1608Metric; Listing https://www.digikey.com/en/products/detail/yageo/RC0402FR-0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 -> https://www.digikey.com/en/products/detail/yageo/RC0603FR-0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
Changed lines of the file:
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@@
 			)
 		)
-		(property "Footprint" "Resistor_SMD:R_0402_1005Metric"
+		(property "Footprint" "Resistor_SMD:R_0603_1608Metric"
 			(at 64.516 128.524 90)
 			(effects
@@
 			)
 		)
-		(property "Listing" "https://www.digikey.com/en/products/detail/yageo/RC0402FR-07330RL/726594"
+		(property "Listing" "https://www.digikey.com/en/products/detail/yageo/RC0603FR-07330RL/727162"
 			(at 63.5 128.27 0)
 			(effects
