File: Project/Controller/XuLabController.kicad_sch (KiCad schematic)
At the start: 4 parts

Commit message: Reorganize pin layout
Other:
- sheet Microcontroller ports: added ADC1_IN13, TIM4_CH4; removed ADC1_IN4, TIM12_CH2
Changed lines of the file:
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@@
 	(title_block
 		(title "Main Sheet")
-		(date "2026-02-10")
+		(date "2026-02-11")
 		(rev "B")
 		(company "CU Boulder Senior Design Team 29 - Xu Lab")
@@
 			)
 		)
-		(pin "TIM12_CH2" output
+		(pin "TIM4_CH4" output
 			(at 165.1 144.78 0)
 			(effects
@@
 			)
 		)
-		(pin "ADC1_IN4" input
+		(pin "ADC1_IN13" input
 			(at 127 115.57 180)
 			(effects

Commit message: Add SHTC3 humidity sensor
Other:
- sheet Sensors ports: added HMD_SCL, HMD_SDA; removed none

Commit message: Change IMU to BMI330
Connections:
- no-connect marks 6 -> 5
Other:
- sheet Sensors ports: added IMU_CS, IMU_INT1, IMU_INT2; removed ACCL_CS, ACCL_INT1, ACCL_INT2, GYRO_CS, GYRO_INT1, GYRO_INT2
