File: Project/Power/Connectors.kicad_sch (KiCad schematic)
At the start: 28 parts, among them J1 Servo, J2 Servo, J3 Servo, J4 Servo, J5 Servo, J6 Servo, J7 Servo, J8 Servo

Commit message: Change connectors to vertical
Parts:
- J1, J2, J3, J4, J5, J6, J7, J8: footprint Connector_JST:JST_VH_S2P-VH_1x02_P3.96mm_Horizontal -> Connector_JST:JST_VH_B2P-VH_1x02_P3.96mm_Vertical; Listing https://www.digikey.com/en/products/detail/jst-sales-america-inc/S2P-VH/9924227 -> https://www.digikey.com/en/products/detail/jst-sales-america-inc/B2P-VH/926547
Changed lines of the file:
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@@
 			)
 		)
-		(property "Footprint" "Connector_JST:JST_VH_S2P-VH_1x02_P3.96mm_Horizontal"
+		(property "Footprint" "Connector_JST:JST_VH_B2P-VH_1x02_P3.96mm_Vertical"
 			(at 212.09 101.6 0)
 			(effects
@@
 			)
 		)
-		(property "Datasheet" "https://mm.digikey.com/Volume0/opasdata/d220001/medias/docus/4886/eVH.doc.pdf"
+		(property "Datasheet" "https://www.jst-mfg.com/product/pdf/eng/eVH.pdf"
 			(at 212.09 101.6 0)
 			(effects
@@
 			)
 		)
-		(property "Listing" "https://www.digikey.com/en/products/detail/jst-sales-america-inc/S2P-VH/9924227"
+		(property "Listing" "https://www.digikey.com/en/products/detail/jst-sales-america-inc/B2P-VH/926547"
 			(at 212.09 101.6 0)
 			(effects
@@
 			)
 		)
-		(property "Footprint" "Connector_JST:JST_VH_S2P-VH_1x02_P3.96mm_Horizontal"
+		(property "Footprint" "Connector_JST:JST_VH_B2P-VH_1x02_P3.96mm_Vertical"
 			(at 212.09 38.1 0)
 			(effects
@@
 			)
 		)
-		(property "Datasheet" "https://mm.digikey.com/Volume0/opasdata/d220001/medias/docus/4886/eVH.doc.pdf"
+		(property "Datasheet" "https://www.jst-mfg.com/product/pdf/eng/eVH.pdf"
 			(at 212.09 38.1 0)
 			(effects
@@
 			)
 		)
-		(property "Listing" "https://www.digikey.com/en/products/detail/jst-sales-america-inc/S2P-VH/9924227"
+		(property "Listing" "https://www.digikey.com/en/products/detail/jst-sales-america-inc/B2P-VH/926547"
 			(at 212.09 38.1 0)
 			(effects
@@
 			)
 		)
-		(property "Footprint" "Connector_JST:JST_VH_S2P-VH_1x02_P3.96mm_Horizontal"
+		(property "Footprint" "Connector_JST:JST_VH_B2P-VH_1x02_P3.96mm_Vertical"
 			(at 123.19 63.5 0)
 			(effects
@@
 			)
 		)
-		(property "Datasheet" "https://mm.digikey.com/Volume0/opasdata/d220001/medias/docus/4886/eVH.doc.pdf"
+		(property "Datasheet" "https://www.jst-mfg.com/product/pdf/eng/eVH.pdf"
 			(at 123.19 63.5 0)
 			(effects
@@
 			)
 		)
-		(property "Listing" "https://www.digikey.com/en/products/detail/jst-sales-america-inc/S2P-VH/9924227"
+		(property "Listing" "https://www.digikey.com/en/products/detail/jst-sales-america-inc/B2P-VH/926547"
 			(at 123.19 63.5 0)
 			(effects
@@
 			)
 		)
-		(property "Footprint" "Connector_JST:JST_VH_S2P-VH_1x02_P3.96mm_Horizontal"
+		(property "Footprint" "Connector_JST:JST_VH_B2P-VH_1x02_P3.96mm_Vertical"
 			(at 123.19 127 0)
 			(effects
@@
 			)
 		)
-		(property "Datasheet" "https://mm.digikey.com/Volume0/opasdata/d220001/medias/docus/4886/eVH.doc.pdf"
+		(property "Datasheet" "https://www.jst-mfg.com/product/pdf/eng/eVH.pdf"
 			(at 123.19 127 0)
 			(effects
@@
 			)
 		)
-		(property "Listing" "https://www.digikey.com/en/products/detail/jst-sales-america-inc/S2P-VH/9924227"
+		(property "Listing" "https://www.digikey.com/en/products/detail/jst-sales-america-inc/B2P-VH/926547"
 			(at 123.19 127 0)
 			(effects
@@
 			)
 		)
-		(property "Footprint" "Connector_JST:JST_VH_S2P-VH_1x02_P3.96mm_Horizontal"
+		(property "Footprint" "Connector_JST:JST_VH_B2P-VH_1x02_P3.96mm_Vertical"
 			(at 123.19 101.6 0)
 			(effects
@@
 			)
 		)
-		(property "Datasheet" "https://mm.digikey.com/Volume0/opasdata/d220001/medias/docus/4886/eVH.doc.pdf"
+		(property "Datasheet" "https://www.jst-mfg.com/product/pdf/eng/eVH.pdf"
 			(at 123.19 101.6 0)
 			(effects
@@
 			)
 		)
-		(property "Listing" "https://www.digikey.com/en/products/detail/jst-sales-america-inc/S2P-VH/9924227"
+		(property "Listing" "https://www.digikey.com/en/products/detail/jst-sales-america-inc/B2P-VH/926547"
 			(at 123.19 101.6 0)
 			(effects
@@
 			)
 		)
-		(property "Footprint" "Connector_JST:JST_VH_S2P-VH_1x02_P3.96mm_Horizontal"
+		(property "Footprint" "Connector_JST:JST_VH_B2P-VH_1x02_P3.96mm_Vertical"
 			(at 212.09 63.5 0)
 			(effects
@@
 			)
 		)
-		(property "Datasheet" "https://mm.digikey.com/Volume0/opasdata/d220001/medias/docus/4886/eVH.doc.pdf"
+		(property "Datasheet" "https://www.jst-mfg.com/product/pdf/eng/eVH.pdf"
 			(at 212.09 63.5 0)
 			(effects
@@
 			)
 		)
-		(property "Listing" "https://www.digikey.com/en/products/detail/jst-sales-america-inc/S2P-VH/9924227"
+		(property "Listing" "https://www.digikey.com/en/products/detail/jst-sales-america-inc/B2P-VH/926547"
 			(at 212.09 63.5 0)
 			(effects
@@
 			)
 		)
-		(property "Footprint" "Connector_JST:JST_VH_S2P-VH_1x02_P3.96mm_Horizontal"
+		(property "Footprint" "Connector_JST:JST_VH_B2P-VH_1x02_P3.96mm_Vertical"
 			(at 123.19 38.1 0)
 			(effects
@@
 			)
 		)
-		(property "Datasheet" "https://mm.digikey.com/Volume0/opasdata/d220001/medias/docus/4886/eVH.doc.pdf"
+		(property "Datasheet" "https://www.jst-mfg.com/product/pdf/eng/eVH.pdf"
 			(at 123.19 38.1 0)
 			(effects
@@
 			)
 		)
-		(property "Listing" "https://www.digikey.com/en/products/detail/jst-sales-america-inc/S2P-VH/9924227"
+		(property "Listing" "https://www.digikey.com/en/products/detail/jst-sales-america-inc/B2P-VH/926547"
 			(at 123.19 38.1 0)
 			(effects
@@
 			)
 		)
-		(property "Footprint" "Connector_JST:JST_VH_S2P-VH_1x02_P3.96mm_Horizontal"
+		(property "Footprint" "Connector_JST:JST_VH_B2P-VH_1x02_P3.96mm_Vertical"
 			(at 212.09 127 0)
 			(effects
@@
 			)
 		)
-		(property "Datasheet" "https://mm.digikey.com/Volume0/opasdata/d220001/medias/docus/4886/eVH.doc.pdf"
+		(property "Datasheet" "https://www.jst-mfg.com/product/pdf/eng/eVH.pdf"
 			(at 212.09 127 0)
 			(effects
@@
 			)
 		)
-		(property "Listing" "https://www.digikey.com/en/products/detail/jst-sales-america-inc/S2P-VH/9924227"
+		(property "Listing" "https://www.digikey.com/en/products/detail/jst-sales-america-inc/B2P-VH/926547"
 			(at 212.09 127 0)
 			(effects
